File: Kicad_LFO_1/Kicad_LFO_1.kicad_pcb (KiCad board)
At the start: 2 copper layers, 100 x 100 mm, 34 parts, among them J101 LFO555, J102 555 Reset, J103 LFO555Charge, J104 Tri, J105 Sine, P101 HEADER_2x5_Doepfer, SW101 LFO Low, U101 LM555, U102 TL072

Commit message: Power settings + Inv net
Parts:
- removed G***: LOGO, AJ:Johansen_engineering_logo_25mm_front_neg5
- removed G*** (x2): LOGO, AJ:Johansen_engineering_logo_15mm
- removed REF**: MountingHole_2.2mm_M2_Pad_Via, MountingHole:MountingHole_2.2mm_M2_Pad_Via
- added C201: 1u, Capacitor_SMD:C_1206_3216Metric_Pad1.42x1.75mm_HandSolder, F.Cu at (76.0, 58.5)
- added C202: 1u, Capacitor_SMD:C_1206_3216Metric_Pad1.42x1.75mm_HandSolder, F.Cu at (84.0, 58.5)
- added D103: LED, LED_SMD:LED_0805_2012Metric_Pad1.15x1.40mm_HandSolder, F.Cu at (60.0, 113.0)
- added D201: LED, LED_SMD:LED_0805_2012Metric_Pad1.15x1.40mm_HandSolder, F.Cu at (85.0, 51.0)
- added J201: In1.1, AJ-Dropbox-Kicad:PJ301SM, F.Cu at (80.0, 72.0)
- added J202: In1.2, AJ-Dropbox-Kicad:PJ301SM, F.Cu at (80.0, 81.0)
- added J203: In1.3, AJ-Dropbox-Kicad:PJ301SM, F.Cu at (80.0, 90.0)
- added J204: Out1, AJ-Dropbox-Kicad:PJ301SM, F.Cu at (80.0, 99.0)
- added J205: In2, AJ-Dropbox-Kicad:PJ301SM, F.Cu at (80.0, 118.0)
- added J206: Out2.1, AJ-Dropbox-Kicad:PJ301SM, F.Cu at (80.0, 127.0)
- added J207: Out2.2, AJ-Dropbox-Kicad:PJ301SM, F.Cu at (80.0, 136.0)
- added J208: Out2.3, AJ-Dropbox-Kicad:PJ301SM, F.Cu at (80.0, 145.0)
- added P201: HEADER_2x5_Doepfer, Connector_IDC:IDC-Header_2x05_P2.54mm_Vertical, B.Cu at (85.0, 56.0)
- added R112: 22k, Resistor_SMD:R_0805_2012Metric_Pad1.15x1.40mm_HandSolder, F.Cu at (58.0, 113.0)
- added R201: 47k, Resistor_SMD:R_0805_2012Metric_Pad1.15x1.40mm_HandSolder, B.Cu at (73.5, 42.0)
- added R202: 20k, Resistor_SMD:R_0805_2012Metric_Pad1.15x1.40mm_HandSolder, B.Cu at (75.9, 45.3)
- added R203: 47k, Resistor_SMD:R_0805_2012Metric_Pad1.15x1.40mm_HandSolder, B.Cu at (68.8, 42.0)
- added R204: 47k, Resistor_SMD:R_0805_2012Metric_Pad1.15x1.40mm_HandSolder, B.Cu at (81.2, 28.4)
- added R205: 47k, Resistor_SMD:R_0805_2012Metric_Pad1.15x1.40mm_HandSolder, B.Cu at (64.0, 42.0)
- added R206: 47k, Resistor_SMD:R_0805_2012Metric_Pad1.15x1.40mm_HandSolder, B.Cu at (97.3, 41.0)
- added R207: 4k7, Resistor_SMD:R_0805_2012Metric_Pad1.15x1.40mm_HandSolder, B.Cu at (78.3, 42.4)
- added R208: 47k, Resistor_SMD:R_0805_2012Metric_Pad1.15x1.40mm_HandSolder, B.Cu at (80.7, 45.3)
- added R209: 20k, Resistor_SMD:R_0805_2012Metric_Pad1.15x1.40mm_HandSolder, B.Cu at (85.4, 45.3)
- added R210: 47k, Resistor_SMD:R_0805_2012Metric_Pad1.15x1.40mm_HandSolder, B.Cu at (83.0, 42.4)
- added R211: 4k7, Resistor_SMD:R_0805_2012Metric_Pad1.15x1.40mm_HandSolder, B.Cu at (87.8, 42.4)
- added R212: 47k, Resistor_SMD:R_0805_2012Metric_Pad1.15x1.40mm_HandSolder, B.Cu at (90.2, 45.3)
- added R213: 4k7, Resistor_SMD:R_0805_2012Metric_Pad1.15x1.40mm_HandSolder, B.Cu at (97.3, 38.1)
- added R214: 4k7, Resistor_SMD:R_0805_2012Metric_Pad1.15x1.40mm_HandSolder, B.Cu at (97.3, 35.1)
- added R215: 22k, Resistor_SMD:R_0805_2012Metric_Pad1.15x1.40mm_HandSolder, F.Cu at (81.0, 51.0)
- added SW201: Inv/NonInv, AJ-Dropbox-Kicad:SP1MS1, F.Cu at (80.0, 62.0)
- added SW202: Inv/NonInv, AJ-Dropbox-Kicad:SP1MS1, F.Cu at (80.0, 109.0)
- added U201: TL082, AJ-Dropbox-Kicad:AJ_SO-8_5.3x6.2mm_P1.27mm, B.Cu at (80.0, 104.0)
Routing:
- net -12VA: track 0.00 -> 53.4 mm
- net +12L: track 0.00 -> 49.6 mm
- net -12V: track 38.3 -> 43.7 mm
- net Net-(D103-Pad2): track 0.00 -> 2.88 mm
Other:
- board text added: "+12v"
- board text added: "-12v"

Commit message: cleanup and decoupl
Parts:
- moved R214 111.6 mm to (78.0, 145.0), turned to 180 degrees
- moved R213 99.8 mm to (78.0, 136.0), turned to 180 degrees
- moved R211 85.2 mm to (78.0, 127.0), turned to 180 degrees
- moved R210 75.6 mm to (82.0, 118.0)
- moved R209 67.3 mm to (82.0, 112.5)
- moved R206 63.3 mm to (87.0, 103.5), turned to 270 degrees
- moved R208 63.0 mm to (87.0, 108.0), turned to 90 degrees
- moved R212 62.9 mm to (73.5, 106.0)
- moved R207 56.6 mm to (78.0, 99.0), turned to 180 degrees
- moved R201 54.7 mm to (87.0, 95.0), turned to 270 degrees
- moved R204 53.3 mm to (72.5, 81.0)
- moved R202 50.2 mm to (83.0, 95.0), turned to 90 degrees
- moved R205 48.7 mm to (72.5, 90.0)
- moved R203 30.2 mm to (72.5, 72.0)
- turned J205 to 270 degrees
Connections:
- net Net-(R201-Pad1) renamed /KicadJE_MMX2/Inv1
- net Net-(R208-Pad1) renamed /KicadJE_MMX2/Inv2
Routing:
- net Net-(R206-Pad2): track 0.00 -> 51.2 mm, vias 0 -> 2
- net Out2: track 0.00 -> 48.6 mm
- net /KicadJE_MMX2/Inv1: track 0.00 -> 48.6 mm
- net GND: track 36.1 -> 83.5 mm, vias 6 -> 8
- net In1: track 0.00 -> 31.8 mm, vias 0 -> 1
- net Net-(J204-PadT): track 0.00 -> 26.1 mm
- net /KicadJE_MMX2/Inv2: track 0.00 -> 16.3 mm
- net Out1: track 0.00 -> 11.4 mm, vias 0 -> 2
- net In2: track 0.00 -> 9.40 mm
- net -12VA: track 53.4 -> 61.5 mm
- net Net-(R212-Pad2): track 0.00 -> 7.00 mm
- net +12L: track 49.6 -> 54.8 mm
- net Net-(D201-Pad2): track 0.00 -> 1.95 mm
- net Net-(J208-PadT): track 0.00 -> 1.89 mm
- net Net-(J207-PadT): track 0.00 -> 1.89 mm
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- added copper zone on B.Cu, net +12L
- added copper zone on B.Cu, net -12VA
