File: Kicad_LFO_1/Kicad_LFO_1.kicad_pcb (KiCad board)
At the start: 2 copper layers, 100 x 100 mm, 139 parts, among them J101 LFO555, J102 555 Reset, J103 LFO555Charge, J104 Tri, J105 Sine, J201 In1.1, J202 In1.2, J203 In1.3, J204 Out1, J205 In2, J206 Out2.1, J207 Out2.2, J208 Out2.3, J302 Tri, J303 LFO_SQ, J304 Sine, J401 NAND_IN1, J402 NAND_OUT, J403 NAND_IN2, J404 AND_IN1, J405 AND_OUT, J406 AND_IN2, J407 NOT_OUT, J408 NOT_IN, J501 FF_In1, J502 FF_In2, J503 FF_Out1, J504 FF_Out2, P101 HEADER_2x5_Doepfer, P201 HEADER_2x5_Doepfer, P301 HEADER_2x5_Doepfer, P401 HEADER_2x5_Doepfer, P501 HEADER_2x5_Doepfer, SW101 LFO Low, SW201 Inv/NonInv, SW202 Inv/NonInv, U101 LM555, U102 TL072, U201 TL082, U301 TL072, U302 TL072, U402 74LS00, U501 4013

Commit message: SMD Placed
Parts:
- added D505: LEDOut1, LED_THT:LED_D3.0mm, F.Cu at (116.8, 145.8)
- added D506: LEDOut2, LED_THT:LED_D3.0mm, F.Cu at (116.8, 102.0)
- added R506: 22k, Resistor_SMD:R_0805_2012Metric_Pad1.15x1.40mm_HandSolder, B.Cu at (116.2, 141.8)
- added R507: 22k, Resistor_SMD:R_0805_2012Metric_Pad1.15x1.40mm_HandSolder, B.Cu at (116.5, 98.0)
- moved R505 106.3 mm to (123.5, 135.2), turned to 270 degrees
- moved R503 88.4 mm to (123.5, 121.2), turned to 270 degrees
- moved D504 87.9 mm to (123.2, 127.2), turned to 270 degrees
- moved U501 75.0 mm to (120.0, 110.8)
- moved R504 61.6 mm to (123.5, 91.5), turned to 90 degrees
- moved R502 57.4 mm to (123.5, 77.5), turned to 90 degrees
- moved D503 46.4 mm to (116.5, 83.5), turned to 270 degrees
- moved C502 45.2 mm to (114.2, 64.5), turned to 90 degrees
- moved D502 42.6 mm to (116.5, 77.8), turned to 270 degrees
- moved C501 34.3 mm to (114.2, 56.8), turned to 90 degrees
- moved R501 33.7 mm to (126.0, 56.8), turned to 90 degrees
- moved D501 16.9 mm to (126.0, 52.5), turned to 90 degrees

Commit message: Update Kicad_LFO_1.kicad_pcb
Parts:
- turned U501 to 270 degrees
Routing:
- net +12V: track 292.7 -> 368.3 mm
- net FF_OUT1: track 0.00 -> 64.5 mm, vias 0 -> 2
- net GND: track 204.6 -> 254.3 mm
- net FF_OUT2: track 0.00 -> 44.1 mm
- net FF_IN1: track 0.00 -> 32.9 mm
- net -12V: track 106.5 -> 128.6 mm
- net Net-(D502-Pad2): track 0.00 -> 10.7 mm
- net Net-(D504-Pad1): track 0.00 -> 8.32 mm
- net FF_IN2: track 0.00 -> 8.27 mm
- net Net-(U501-Pad12): track 0.00 -> 5.23 mm
- net Net-(U501-Pad2): track 0.00 -> 5.23 mm
- net Net-(D501-Pad2): track 0.00 -> 5.10 mm
- net Net-(J504-PadT): track 0.00 -> 4.89 mm
- net Net-(D506-Pad2): track 0.00 -> 3.92 mm
- net Net-(D505-Pad2): track 0.00 -> 3.82 mm
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
Commit message: Copper plane
Routing:
- net GND: track 254.3 -> 299.6 mm, vias 16 -> 20
- net +12V: track 368.3 -> 396.1 mm, vias 5 -> 6
Changed lines of the file:
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@@
     (thickness 1.6)
     (drawings 33)
-    (tracks 852)
+    (tracks 872)
     (zones 0)
     (modules 143)
@@
   (segment (start 72.475 107.525) (end 72 108) (width 0.4) (layer B.Cu) (net 1))
   (segment (start 59.809999 56.286001) (end 58.81 57.286) (width 0.4) (layer F.Cu) (net 1))
-  (segment (start 65.67099 50.42501) (end 59.809999 56.286001) (width 0.4) (layer F.Cu) (net 1))
-  (segment (start 74.34501 50.42501) (end 65.67099 50.42501) (width 0.4) (layer F.Cu) (net 1))
+  (segment (start 65.67099 50.42501) (end 59.809999 56.286001) (width 0.2) (layer F.Cu) (net 1))
+  (segment (start 74.34501 50.42501) (end 65.67099 50.42501) (width 0.2) (layer F.Cu) (net 1))
   (segment (start 77.38 53.46) (end 74.34501 50.42501) (width 0.4) (layer F.Cu) (net 1))
   (segment (start 79.92 52.945) (end 79.92 53.46) (width 0.4) (layer F.Cu) (net 1))
@@
   (segment (start 119.98 145.75) (end 120 145.73) (width 0.4) (layer B.Cu) (net 1))
   (segment (start 116.75 145.75) (end 119.98 145.75) (width 0.4) (layer B.Cu) (net 1))
+  (via (at 125 107.25) (size 1) (drill 0.5) (layers F.Cu B.Cu) (net 1))
+  (segment (start 123.81 108) (end 124.25 108) (width 0.4) (layer B.Cu) (net 1))
+  (segment (start 124.25 108) (end 125 107.25) (width 0.4) (layer B.Cu) (net 1))
+  (via (at 124.42501 115.25) (size 1) (drill 0.5) (layers F.Cu B.Cu) (net 1))
+  (segment (start 123.81 113.4) (end 123.81 114.63499) (width 0.4) (layer B.Cu) (net 1))
+  (segment (start 123.81 114.63499) (end 124.42501 115.25) (width 0.4) (layer B.Cu) (net 1))
+  (via (at 132.25 57.75) (size 1) (drill 0.5) (layers F.Cu B.Cu) (net 1))
+  (segment (start 121.29 57.88) (end 132.62 57.88) (width 0.2) (layer F.Cu) (net 1))
+  (segment (start 132.62 57.88) (end 132.75 57.75) (width 0.4) (layer F.Cu) (net 1))
+  (segment (start 118.75 57.88) (end 101.54 57.88) (width 0.2) (layer F.Cu) (net 1))
+  (via (at 87 60.25) (size 1) (drill 0.5) (layers F.Cu B.Cu) (net 1))
+  (segment (start 99 57.88) (end 89.37 57.88) (width 0.2) (layer F.Cu) (net 1))
+  (segment (start 89.37 57.88) (end 87 60.25) (width 0.2) (layer F.Cu) (net 1))
   (segment (start 62.595 66.62) (end 62.5 66.525) (width 0.25) (layer B.Cu) (net 2))
   (segment (start 62.595 69.2) (end 62.595 66.62) (width 0.25) (layer B.Cu) (net 2))
@@
   (segment (start 112.6 57.5) (end 112.6 74.7) (width 0.6) (layer B.Cu) (net 6))
   (segment (start 112.6 74.7) (end 112.6 109) (width 0.6) (layer B.Cu) (net 6))
+  (segment (start 101.6175 55.2625) (end 101.54 55.34) (width 0.4) (layer B.Cu) (net 6))
+  (segment (start 114.25 55.2625) (end 101.6175 55.2625) (width 0.2) (layer B.Cu) (net 6))
+  (segment (start 124.908696 50.49999) (end 131.49999 50.49999) (width 0.2) (layer B.Cu) (net 6))
+  (segment (start 121.29 55.34) (end 121.29 54.118686) (width 0.4) (layer B.Cu) (net 6))
+  (segment (start 121.29 54.118686) (end 124.908696 50.49999) (width 0.2) (layer B.Cu) (net 6))
+  (via (at 133 52) (size 1) (drill 0.5) (layers F.Cu B.Cu) (net 6))
+  (segment (start 131.49999 50.49999) (end 133 52) (width 0.2) (layer B.Cu) (net 6))
   (segment (start 64 75.935) (end 63.865 75.8) (width 0.25) (layer B.Cu) (net 7))
   (segment (start 64 78.975) (end 64 75.935) (width 0.25) (layer B.Cu) (net 7))
@@
       )
     )
+  )
+  (zone (net 1) (net_name GND) (layer F.Cu) (hatch edge 0.508)
+    (connect_pads (clearance 0.508))
+    (min_thickness 0.254)
+    (fill yes (arc_segments 32) (thermal_gap 0.508) (thermal_bridge_width 0.508))
+    (polygon
+      (pts
+        (xy 112 51) (xy 128 51) (xy 128 149) (xy 112 149)
+      )
+    )
+  )
+  (zone (net 6) (net_name +12V) (layer B.Cu) (hatch edge 0.508)
+    (connect_pads (clearance 0.508))
+    (min_thickness 0.254)
+    (fill yes (arc_segments 32) (thermal_gap 0.508) (thermal_bridge_width 0.508))
+    (polygon
+      (pts
+        (xy 112 51) (xy 128 51) (xy 128 149) (xy 112 149)
+      )
+    )

Commit message: Update Kicad_LFO_1.kicad_pcb
Parts:
- added G***: LOGO, AJ:Johansen_engineering_logo_15mm, B.Cu at (113.5, 125.8)
Other:
- board text added: "FLIP FLOP"
- board text added: "FlipFlop Johansen Engineering 2019/04/16 - Rev A"
- board text added: "MMX2"
- board text added: "NAND"
- board text added: "NAND Johansen Engineering 2019/04/15 - Rev A"

Commit message: gerber
Routing:
- net +12V: track 396.1 -> 440.5 mm, vias 6 -> 11
- net (no net): track 0.00 -> 5.23 mm, vias 0 -> 2
- net GND: track 299.6 -> 301.7 mm, vias 20 -> 21
Changed lines of the file:
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@@
     (thickness 1.6)
     (drawings 38)
-    (tracks 872)
+    (tracks 902)
     (zones 0)
     (modules 144)
@@
       (layerselection 0x010fc_ffffffff)
       (usegerberextensions false)
-      (usegerberattributes false)
+      (usegerberattributes true)
       (usegerberadvancedattributes false)
       (creategerberjobfile false)
-      (excludeedgelayer true)
-      (linewidth 0.100000)
+      (excludeedgelayer false)
+      (linewidth 0.150000)
       (plotframeref false)
       (viasonmask false)
@@
       (outputformat 1)
       (mirror false)
-      (drillshape 1)
+      (drillshape 0)
       (scaleselection 1)
-      (outputdirectory ""))
+      (outputdirectory "gerber_revA"))
   )
   (net 0 "")
@@
   (gr_line (start 50 150) (end 150 150) (layer Edge.Cuts) (width 0.05))
   (gr_line (start 50 50) (end 50 150) (layer Edge.Cuts) (width 0.05))
+  (via (at 136.5 76.375) (size 0.8) (drill 0.4) (layers F.Cu B.Cu) (net 0))
+  (segment (start 136.75 76.25) (end 136.625 76.25) (width 0.25) (layer B.Cu) (net 0))
+  (segment (start 136.625 76.25) (end 136.5 76.375) (width 0.25) (layer B.Cu) (net 0))
+  (via (at 136.75 71.55) (size 0.8) (drill 0.4) (layers F.Cu B.Cu) (net 0))
+  (segment (start 136.5 76.375) (end 136.5 71.8) (width 0.25) (layer F.Cu) (net 0))
+  (segment (start 136.5 71.8) (end 136.75 71.55) (width 0.25) (layer F.Cu) (net 0))
   (segment (start 62.6075 109.88) (end 62 110.4875) (width 0.4) (layer B.Cu) (net 1))
   (segment (start 67 109.88) (end 62.6075 109.88) (width 0.4) (layer B.Cu) (net 1))
@@
   (segment (start 99 57.88) (end 89.37 57.88) (width 0.2) (layer F.Cu) (net 1))
   (segment (start 89.37 57.88) (end 87 60.25) (width 0.2) (layer F.Cu) (net 1))
+  (segment (start 133.55 108) (end 132.8 108.75) (width 0.4) (layer B.Cu) (net 1))
+  (segment (start 134.225 108) (end 133.55 108) (width 0.4) (layer B.Cu) (net 1))
+  (via (at 132.5 108.75) (size 1) (drill 0.5) (layers F.Cu B.Cu) (net 1))
+  (segment (start 132.8 108.75) (end 132.5 108.75) (width 0.4) (layer B.Cu) (net 1))
   (segment (start 62.595 66.62) (end 62.5 66.525) (width 0.25) (layer B.Cu) (net 2))
   (segment (start 62.595 69.2) (end 62.595 66.62) (width 0.25) (layer B.Cu) (net 2))
@@
   (segment (start 101.54 55.34) (end 94.3275 55.34) (width 0.6) (layer B.Cu) (net 6))
   (segment (start 102.9 91.06) (end 102.45 91.06) (width 0.4) (layer B.Cu) (net 6))
-  (segment (start 105 88.96) (end 102.9 91.06) (width 0.6) (layer B.Cu) (net 6))
-  (segment (start 105 58.8) (end 105 88.96) (width 0.6) (layer B.Cu) (net 6))
-  (segment (start 101.54 55.34) (end 105 58.8) (width 0.6) (layer B.Cu) (net 6))
   (segment (start 95.2 133.5) (end 95.2 132.5) (width 0.4) (layer B.Cu) (net 6))
   (segment (start 93.92999 134.77001) (end 95.2 133.5) (width 0.4) (layer B.Cu) (net 6))
@@
   (segment (start 144.905 96.8325) (end 146.4875 95.25) (width 0.4) (layer B.Cu) (net 6))
   (segment (start 144.905 98.2) (end 144.905 96.8325) (width 0.4) (layer B.Cu) (net 6))
-  (segment (start 146.405 78.8325) (end 146.4875 78.75) (width 0.4) (layer B.Cu) (net 6))
-  (segment (start 146.405 81.7) (end 146.405 78.8325) (width 0.4) (layer B.Cu) (net 6))
   (segment (start 136.859999 93.199999) (end 144.437499 93.199999) (width 0.4) (layer B.Cu) (net 6))
   (segment (start 136.5 92.84) (end 136.859999 93.199999) (width 0.4) (layer B.Cu) (net 6))
@@
   (via (at 133 52) (size 1) (drill 0.5) (layers F.Cu B.Cu) (net 6))
   (segment (start 131.49999 50.49999) (end 133 52) (width 0.2) (layer B.Cu) (net 6))
+  (segment (start 103.44 91.06) (end 102.9 91.06) (width 0.6) (layer B.Cu) (net 6))
+  (segment (start 105 89.5) (end 103.44 91.06) (width 0.6) (layer B.Cu) (net 6))
+  (segment (start 101.54 55.34) (end 105 58.8) (width 0.6) (layer B.Cu) (net 6))
+  (segment (start 105 58.8) (end 105 89.5) (width 0.6) (layer B.Cu) (net 6))
+  (segment (start 146.4875 81.6175) (end 146.405 81.7) (width 0.4) (layer B.Cu) (net 6))
+  (segment (start 146.4875 78.75) (end 146.4875 81.6175) (width 0.4) (layer B.Cu) (net 6))
+  (via (at 134.25 90.400002) (size 1) (drill 0.5) (layers F.Cu B.Cu) (net 6))
+  (segment (start 133.96 92.84) (end 133.96 90.690002) (width 0.4) (layer F.Cu) (net 6))
+  (segment (start 133.96 90.690002) (end 134.25 90.400002) (width 0.4) (layer F.Cu) (net 6))
+  (via (at 134.679136 85.320864) (size 1) (drill 0.5) (layers F.Cu B.Cu) (net 6))
+  (segment (start 134.25 90.400002) (end 134.25 85.75) (width 0.4) (layer B.Cu) (net 6))
+  (segment (start 134.25 85.75) (end 134.679136 85.320864) (width 0.4) (layer B.Cu) (net 6))
+  (via (at 135.595864 83.904136) (size 1) (drill 0.5) (layers F.Cu B.Cu) (net 6))
+  (segment (start 134.679136 85.320864) (end 134.679136 84.820864) (width 0.4) (layer F.Cu) (net 6))
+  (segment (start 134.679136 84.820864) (end 135.595864 83.904136) (width 0.4) (layer F.Cu) (net 6))
+  (via (at 134.25 81.5) (size 1) (drill 0.5) (layers F.Cu B.Cu) (net 6))
+  (segment (start 135.595864 83.904136) (end 135.595864 82.845864) (width 0.4) (layer B.Cu) (net 6))
+  (segment (start 135.595864 82.845864) (end 134.25 81.5) (width 0.4) (layer B.Cu) (net 6))
+  (segment (start 134.25 81.5) (end 133.542894 81.5) (width 0.4) (layer F.Cu) (net 6))
+  (segment (start 133.542894 81.5) (end 132 81.5) (width 0.4) (layer F.Cu) (net 6))
+  (via (at 132.5 110.25) (size 1) (drill 0.5) (layers F.Cu B.Cu) (net 6))
+  (segment (start 131.599999 109.349999) (end 132.5 110.25) (width 0.4) (layer F.Cu) (net 6))
+  (segment (start 132 81.5) (end 131.599999 81.900001) (width 0.4) (layer F.Cu) (net 6))
+  (segment (start 131.599999 81.900001) (end 131.599999 109.349999) (width 0.4) (layer F.Cu) (net 6))
   (segment (start 64 75.935) (end 63.865 75.8) (width 0.25) (layer B.Cu) (net 7))
   (segment (start 64 78.975) (end 64 75.935) (width 0.25) (layer B.Cu) (net 7))
@@
   (segment (start 67.576397 127.576397) (end 67.576397 136.423603) (width 0.4) (layer B.Cu) (net 9))
   (segment (start 67.576397 136.423603) (end 62 142) (width 0.4) (layer B.Cu) (net 9))
-  (segment (start 63.475 117.5) (end 63.96 117.5) (width 0.4) (layer F.Cu) (net 9))
-  (segment (start 60 114.025) (end 63.475 117.5) (width 0.4) (layer F.Cu) (net 9))
   (segment (start 101.54 65.5) (end 99 65.5) (width 0.4) (layer B.Cu) (net 9))
   (segment (start 98.812501 65.312501) (end 99 65.5) (width 0.4) (layer B.Cu) (net 9))
@@
   (segment (start 114.7375 65.5) (end 114.25 65.9875) (width 0.4) (layer B.Cu) (net 9))
   (segment (start 118.75 65.5) (end 114.7375 65.5) (width 0.4) (layer B.Cu) (net 9))
+  (segment (start 63 117.5) (end 63.96 117.5) (width 0.4) (layer F.Cu) (net 9))
+  (segment (start 60 114.025) (end 60 114.5) (width 0.4) (layer F.Cu) (net 9))
+  (segment (start 60 114.5) (end 63 117.5) (width 0.4) (layer F.Cu) (net 9))
   (segment (start 51.19 83.125787) (end 51.19 79.46) (width 0.25) (layer B.Cu) (net 10))
   (segment (start 51.19 84.54) (end 51.19 83.125787) (width 0.25) (layer B.Cu) (net 10))

Commit message: RevB PCB
Connections:
- J401 pad TN: GND -> +12V
- J403 pad TN: GND -> +12V
- J404 pad TN: GND -> +12V
- J406 pad TN: GND -> +12V
Routing:
- net GND: track 301.7 -> 306.6 mm
Changed lines of the file:
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@@
     (thickness 1.6)
     (drawings 38)
-    (tracks 902)
+    (tracks 906)
     (zones 0)
     (modules 144)
@@
       (drillshape 0)
       (scaleselection 1)
-      (outputdirectory "gerber_revA"))
+      (outputdirectory "gerber_revB"))
   )
   (net 0 "")
@@
     (fp_circle (center 0 0) (end 1.8 0) (layer F.SilkS) (width 0.15))
     (pad TN thru_hole oval (at 0 3.38 90) (size 2.8 1.6) (drill oval 2 0.6) (layers *.Cu *.Mask)
-      (net 1 GND))
+      (net 6 +12V))
     (pad S thru_hole oval (at 0 6.48 90) (size 2.4 1.6) (drill oval 1.4 0.6) (layers *.Cu *.Mask)
       (net 1 GND))
@@
       (net 1 GND))
     (pad TN thru_hole oval (at 0 3.38 90) (size 2.8 1.6) (drill oval 2 0.6) (layers *.Cu *.Mask)
-      (net 1 GND))
+      (net 6 +12V))
     (model ${KIPRJMOD}/Local.pretty/PJ398SM.step
       (offset (xyz 0 0 9))
@@
       (net 1 GND))
     (pad TN thru_hole oval (at 0 3.38 90) (size 2.8 1.6) (drill oval 2 0.6) (layers *.Cu *.Mask)
-      (net 1 GND))
+      (net 6 +12V))
     (model ${KIPRJMOD}/Local.pretty/PJ398SM.step
       (offset (xyz 0 0 9))
@@
     (fp_circle (center 0 0) (end 1.8 0) (layer F.SilkS) (width 0.15))
     (pad TN thru_hole oval (at 0 3.38 90) (size 2.8 1.6) (drill oval 2 0.6) (layers *.Cu *.Mask)
-      (net 1 GND))
+      (net 6 +12V))
     (pad S thru_hole oval (at 0 6.48 90) (size 2.4 1.6) (drill oval 1.4 0.6) (layers *.Cu *.Mask)
       (net 1 GND))
@@
   (segment (start 103.4 80.205001) (end 103.355001 80.25) (width 0.4) (layer B.Cu) (net 1))
   (segment (start 103.4 75.5) (end 103.4 80.205001) (width 0.4) (layer B.Cu) (net 1))
-  (segment (start 103.4 104.955001) (end 103.355001 105) (width 0.4) (layer B.Cu) (net 1))
-  (segment (start 103.4 101.75) (end 103.4 104.955001) (width 0.4) (layer B.Cu) (net 1))
-  (segment (start 103.505001 113.874999) (end 103.38 114) (width 0.4) (layer B.Cu) (net 1))
-  (segment (start 103.505001 111) (end 103.505001 113.874999) (width 0.4) (layer B.Cu) (net 1))
-  (segment (start 103.355001 141.544999) (end 103.4 141.5) (width 0.4) (layer B.Cu) (net 1))
-  (segment (start 103.355001 145) (end 103.355001 141.544999) (width 0.4) (layer B.Cu) (net 1))
-  (segment (start 103.505001 135.799998) (end 103.38 135.924999) (width 0.4) (layer B.Cu) (net 1))
-  (segment (start 103.505001 132.474999) (end 103.505001 135.799998) (width 0.4) (layer B.Cu) (net 1))
   (via (at 95 83) (size 1) (drill 0.5) (layers F.Cu B.Cu) (net 1))
   (segment (start 97.05 83.44) (end 95.44 83.44) (width 0.4) (layer B.Cu) (net 1))
@@
   (via (at 132.5 108.75) (size 1) (drill 0.5) (layers F.Cu B.Cu) (net 1))
   (segment (start 132.8 108.75) (end 132.5 108.75) (width 0.4) (layer B.Cu) (net 1))
+  (segment (start 106.455001 104.955001) (end 106.455001 105) (width 0.4) (layer B.Cu) (net 1))
+  (segment (start 103.4 101.9) (end 106.455001 104.955001) (width 0.4) (layer B.Cu) (net 1))
+  (segment (start 103.4 101.75) (end 103.4 101.9) (width 0.4) (layer B.Cu) (net 1))
+  (segment (start 106.355001 114) (end 106.48 114) (width 0.4) (layer B.Cu) (net 1))
+  (segment (start 103.505001 111.15) (end 106.355001 114) (width 0.4) (layer B.Cu) (net 1))
+  (segment (start 103.505001 111) (end 103.505001 111.15) (width 0.4) (layer B.Cu) (net 1))
+  (segment (start 106.48 135.599998) (end 106.48 135.924999) (width 0.4) (layer B.Cu) (net 1))
+  (segment (start 103.505001 132.624999) (end 106.48 135.599998) (width 0.4) (layer B.Cu) (net 1))
+  (segment (start 103.505001 132.474999) (end 103.505001 132.624999) (width 0.4) (layer B.Cu) (net 1))
+  (segment (start 106.455001 144.705001) (end 106.455001 145) (width 0.4) (layer B.Cu) (net 1))
+  (segment (start 103.4 141.65) (end 106.455001 144.705001) (width 0.4) (layer B.Cu) (net 1))
+  (segment (start 103.4 141.5) (end 103.4 141.65) (width 0.4) (layer B.Cu) (net 1))
   (segment (start 62.595 66.62) (end 62.5 66.525) (width 0.25) (layer B.Cu) (net 2))
   (segment (start 62.595 69.2) (end 62.595 66.62) (width 0.25) (layer B.Cu) (net 2))

Commit message: Update Kicad_LFO_1.kicad_pcb
Routing:
- net -12V: track 128.9 -> 254.6 mm, vias 2 -> 4
Changed lines of the file:
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@@
     (thickness 1.6)
     (drawings 38)
-    (tracks 906)
+    (tracks 916)
     (zones 0)
     (modules 144)
@@
   (segment (start 60 114.025) (end 60 114.5) (width 0.4) (layer F.Cu) (net 9))
   (segment (start 60 114.5) (end 63 117.5) (width 0.4) (layer F.Cu) (net 9))
+  (segment (start 67.576397 148.423603) (end 68.402794 149.25) (width 0.2) (layer B.Cu) (net 9))
+  (segment (start 67.576397 136.423603) (end 67.576397 148.423603) (width 0.2) (layer B.Cu) (net 9))
+  (segment (start 68.402794 149.25) (end 132.25 149.25) (width 0.2) (layer B.Cu) (net 9))
+  (segment (start 132.25 149.25) (end 132.25 124.5) (width 0.2) (layer B.Cu) (net 9))
+  (via (at 134.64999 124.5) (size 0.8) (drill 0.4) (layers F.Cu B.Cu) (net 9))
+  (segment (start 132.25 124.5) (end 134.64999 124.5) (width 0.2) (layer B.Cu) (net 9))
+  (via (at 136.09999 124.5) (size 0.8) (drill 0.4) (layers F.Cu B.Cu) (net 9))
+  (segment (start 134.64999 124.5) (end 136.09999 124.5) (width 0.2) (layer F.Cu) (net 9))
+  (segment (start 136.09999 114.91251) (end 143.5125 107.5) (width 0.2) (layer B.Cu) (net 9))
+  (segment (start 136.09999 124.5) (end 136.09999 114.91251) (width 0.2) (layer B.Cu) (net 9))
   (segment (start 51.19 83.125787) (end 51.19 79.46) (width 0.25) (layer B.Cu) (net 10))
   (segment (start 51.19 84.54) (end 51.19 83.125787) (width 0.25) (layer B.Cu) (net 10))
