File: Kicad_LFO_1_2/Kicad_LFO_1_2.kicad_pcb (KiCad board)
At the start: 2 copper layers, 100 x 100 mm, 144 parts, among them J101 LFO555, J102 555 Reset, J103 LFO555Charge, J104 Tri, J105 Sine, J201 In1.1, J202 In1.2, J203 In1.3, J204 Out1, J205 In2, J206 Out2.1, J207 Out2.2, J208 Out2.3, J302 Tri, J303 LFO_SQ, J304 Sine, J401 NAND_IN1, J402 NAND_OUT, J403 NAND_IN2, J404 AND_IN1, J405 AND_OUT, J406 AND_IN2, J407 NOT_OUT, J408 NOT_IN, J501 FF_In1, J502 FF_In2, J503 FF_Out1, J504 FF_Out2, P101 HEADER_2x5_Doepfer, P201 HEADER_2x5_Doepfer, P301 HEADER_2x5_Doepfer, P401 HEADER_2x5_Doepfer, P501 HEADER_2x5_Doepfer, SW101 LFO Low, SW201 Inv/NonInv, SW202 Inv/NonInv, U101 LM555, U102 TL072, U201 TL082, U301 TL072, U302 TL072, U402 74LS00, U501 4013

Commit message: LED's swapped for flip flop
Parts:
- moved R506 43.8 mm to (114.2, 98.0)
- moved R507 43.8 mm to (116.2, 141.8)
- moved D505 43.8 mm to (116.8, 102.0)
- moved D506 43.8 mm to (116.8, 145.8)
Routing:
- net FF_OUT2: track 44.1 -> 38.4 mm
- net Net-(D505-Pad2): track 3.82 -> 2.99 mm
Changed lines of the file:
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@@
     (thickness 1.6)
     (drawings 38)
-    (tracks 916)
+    (tracks 917)
     (zones 0)
     (modules 144)
@@
   )
   (module LED_THT:LED_D3.0mm (layer F.Cu)
-    (at 116.75 145.75 180)
+    (at 116.75 102 180)
     (descr "LED, diameter 3.0mm, 2 pins")
     (tags "LED diameter 3.0mm 2 pins")
@@
   )
   (module LED_THT:LED_D3.0mm (layer F.Cu)
-    (at 116.75 102 180)
+    (at 116.75 145.75 180)
     (descr "LED, diameter 3.0mm, 2 pins")
     (tags "LED diameter 3.0mm 2 pins")
@@
   )
   (module Resistor_SMD:R_0805_2012Metric_Pad1.15x1.40mm_HandSolder (layer B.Cu)
-    (at 116.25 141.75 270)
+    (at 114.25 98 270)
     (descr "Resistor SMD 0805 (2012 Metric), square (rectangular) end terminal, IPC_7351 nominal with elongated pad for handsoldering. (Body size source: https://docs.google.com/spreadsheets/d/1BsfQQcO9C6DZCsRaXUlFlo91Tg2WpOkGARC1WS5S8t0/edit?usp=sharing), generated with kicad-footprint-generator")
     (tags "resistor handsolder")
@@
   )
   (module Resistor_SMD:R_0805_2012Metric_Pad1.15x1.40mm_HandSolder (layer B.Cu)
-    (at 116.5 98 270)
+    (at 116.25 141.75 270)
     (descr "Resistor SMD 0805 (2012 Metric), square (rectangular) end terminal, IPC_7351 nominal with elongated pad for handsoldering. (Body size source: https://docs.google.com/spreadsheets/d/1BsfQQcO9C6DZCsRaXUlFlo91Tg2WpOkGARC1WS5S8t0/edit?usp=sharing), generated with kicad-footprint-generator")
     (tags "resistor handsolder")
@@
   (segment (start 120 121.33) (end 120.945 122.275) (width 0.25) (layer B.Cu) (net 64))
   (segment (start 120 120.33) (end 120 121.33) (width 0.25) (layer B.Cu) (net 64))
-  (segment (start 123.5 93.2) (end 123.5 92.525) (width 0.25) (layer B.Cu) (net 65))
-  (segment (start 123.5 100.471004) (end 123.5 93.2) (width 0.25) (layer B.Cu) (net 65))
-  (segment (start 120.865994 103.10501) (end 123.5 100.471004) (width 0.25) (layer B.Cu) (net 65))
-  (segment (start 120.086398 103.10501) (end 120.865994 103.10501) (width 0.25) (layer B.Cu) (net 65))
-  (segment (start 116.19 107.001408) (end 120.086398 103.10501) (width 0.25) (layer B.Cu) (net 65))
-  (segment (start 116.19 108) (end 116.19 107.001408) (width 0.25) (layer B.Cu) (net 65))
   (via (at 125.25001 127.6) (size 0.8) (drill 0.4) (layers F.Cu B.Cu) (net 65))
   (segment (start 125.25001 113.205008) (end 125.25001 127.6) (width 0.25) (layer B.Cu) (net 65))
@@
   (segment (start 123.5 127.7) (end 120.93 127.7) (width 0.25) (layer B.Cu) (net 65))
   (segment (start 119.4 128.63) (end 120 128.63) (width 0.25) (layer B.Cu) (net 65))
-  (segment (start 116.25 131.78) (end 119.4 128.63) (width 0.25) (layer B.Cu) (net 65))
-  (segment (start 116.25 140.725) (end 116.25 131.78) (width 0.25) (layer B.Cu) (net 65))
+  (segment (start 123.5 96) (end 123.5 92.525) (width 0.25) (layer B.Cu) (net 65))
+  (segment (start 122.75 96.75) (end 123.5 96) (width 0.25) (layer B.Cu) (net 65))
+  (segment (start 114.25 96.975) (end 114.475 96.75) (width 0.25) (layer B.Cu) (net 65))
+  (segment (start 114.475 96.75) (end 122.75 96.75) (width 0.25) (layer B.Cu) (net 65))
+  (segment (start 123.5 93.2) (end 123.5 92.525) (width 0.25) (layer B.Cu) (net 65))
+  (segment (start 123.5 101) (end 123.5 93.2) (width 0.25) (layer B.Cu) (net 65))
+  (segment (start 118 106.5) (end 123.5 101) (width 0.25) (layer B.Cu) (net 65))
+  (segment (start 116.691408 106.5) (end 118 106.5) (width 0.25) (layer B.Cu) (net 65))
+  (segment (start 116.19 108) (end 116.19 107.001408) (width 0.25) (layer B.Cu) (net 65))
+  (segment (start 116.19 107.001408) (end 116.691408 106.5) (width 0.25) (layer B.Cu) (net 65))
   (segment (start 123.395 90.58) (end 123.5 90.475) (width 0.25) (layer B.Cu) (net 66))
   (segment (start 120 90.58) (end 123.395 90.58) (width 0.25) (layer B.Cu) (net 66))
@@
   (segment (start 120 116.725) (end 123.5 120.225) (width 0.25) (layer B.Cu) (net 69))
   (segment (start 120 113.4) (end 120 116.725) (width 0.25) (layer B.Cu) (net 69))
-  (segment (start 115.2 110.69) (end 117.46 112.95) (width 0.25) (layer B.Cu) (net 70))
-  (segment (start 115.2 107.354998) (end 115.2 110.69) (width 0.25) (layer B.Cu) (net 70))
-  (segment (start 117.975001 104.579997) (end 115.2 107.354998) (width 0.25) (layer B.Cu) (net 70))
-  (segment (start 117.975001 98.911811) (end 117.975001 104.579997) (width 0.25) (layer B.Cu) (net 70))
-  (segment (start 116.5 97.43681) (end 117.975001 98.911811) (width 0.25) (layer B.Cu) (net 70))
   (segment (start 117.46 112.95) (end 117.46 113.4) (width 0.25) (layer B.Cu) (net 70))
-  (segment (start 116.5 96.975) (end 116.5 97.43681) (width 0.25) (layer B.Cu) (net 70))
   (segment (start 124.52501 133.19999) (end 124.123372 133.601628) (width 0.25) (layer B.Cu) (net 70))
   (segment (start 124.52501 121.71182) (end 124.52501 133.19999) (width 0.25) (layer B.Cu) (net 70))
@@
   (segment (start 117.46 114.82141) (end 122.47499 119.8364) (width 0.25) (layer B.Cu) (net 70))
   (segment (start 117.46 113.4) (end 117.46 114.82141) (width 0.25) (layer B.Cu) (net 70))
+  (segment (start 124.123372 134.848372) (end 123.5 134.225) (width 0.25) (layer B.Cu) (net 70))
+  (segment (start 124.52501 135.25001) (end 124.123372 134.848372) (width 0.25) (layer B.Cu) (net 70))
+  (segment (start 124.52501 136.83818) (end 124.52501 135.25001) (width 0.25) (layer B.Cu) (net 70))
+  (segment (start 120.63819 140.725) (end 124.52501 136.83818) (width 0.25) (layer B.Cu) (net 70))
+  (segment (start 116.25 140.725) (end 120.63819 140.725) (width 0.25) (layer B.Cu) (net 70))
   (segment (start 121.27 108.45) (end 121.27 108) (width 0.25) (layer B.Cu) (net 71))
   (segment (start 120.644999 109.075001) (end 121.27 108.45) (width 0.25) (layer B.Cu) (net 71))
@@
   (segment (start 118.73 112.95) (end 119.355001 112.324999) (width 0.25) (layer B.Cu) (net 72))
   (segment (start 118.73 113.4) (end 118.73 112.95) (width 0.25) (layer B.Cu) (net 72))
-  (segment (start 116.25 143.71) (end 116.25 142.775) (width 0.25) (layer B.Cu) (net 73))
-  (segment (start 114.21 145.75) (end 116.25 143.71) (width 0.25) (layer B.Cu) (net 73))
-  (segment (start 116.5 99.71) (end 116.5 99.025) (width 0.25) (layer B.Cu) (net 74))
-  (segment (start 114.21 102) (end 116.5 99.71) (width 0.25) (layer B.Cu) (net 74))
+  (segment (start 116.25 143.71) (end 116.25 142.775) (width 0.25) (layer B.Cu) (net 74))
+  (segment (start 114.21 145.75) (end 116.25 143.71) (width 0.25) (layer B.Cu) (net 74))
+  (segment (start 114.21 99.065) (end 114.25 99.025) (width 0.25) (layer B.Cu) (net 73))
+  (segment (start 114.21 102) (end 114.21 99.065) (width 0.25) (layer B.Cu) (net 73))
   (zone (net 1) (net_name GND) (layer F.Cu) (hatch edge 0.508)
     (connect_pads (clearance 0.508))

Commit message: LFO 1 Routed and labeled
Parts:
- removed G*** (x6): LOGO, AJ:Johansen_engineering_logo_15mm
- removed G***: LOGO, AJ:Johansen_engineering_logo_25mm_front_neg5
- removed RV102: 10k Sine, Potentiometer_THT:Potentiometer_Alps_RK163_Single_Horizontal
- removed RV302: 100k Freq, Potentiometer_THT:Potentiometer_Alps_RK163_Single_Horizontal
- removed U402: 74LS00, Package_SO:SOIC-14_3.9x8.7mm_P1.27mm
- added R113: 470r, Resistor_SMD:R_0805_2012Metric_Pad1.15x1.40mm_HandSolder, F.Cu at (74.4, 39.6)
- added R114: 100r, Resistor_SMD:R_0805_2012Metric_Pad1.15x1.40mm_HandSolder, F.Cu at (74.4, 42.5)
- added R115: 100r, Resistor_SMD:R_0805_2012Metric_Pad1.15x1.40mm_HandSolder, F.Cu at (79.1, 39.6)
- added R116: 100r, Resistor_SMD:R_0805_2012Metric_Pad1.15x1.40mm_HandSolder, F.Cu at (79.1, 42.5)
- added R117: 4k7, Resistor_SMD:R_0805_2012Metric_Pad1.15x1.40mm_HandSolder, F.Cu at (83.9, 39.6)
- added R313: 4k7, Resistor_SMD:R_0805_2012Metric_Pad1.15x1.40mm_HandSolder, B.Cu at (140.2, 128.2)
- added R314: OPEN, Resistor_SMD:R_0805_2012Metric_Pad1.15x1.40mm_HandSolder, B.Cu at (140.2, 89.2)
- added R315: 1k, Resistor_SMD:R_0805_2012Metric_Pad1.15x1.40mm_HandSolder, B.Cu at (144.8, 89.2)
- added R316: 1k, Resistor_SMD:R_0805_2012Metric_Pad1.15x1.40mm_HandSolder, B.Cu at (144.2, 55.2)
- added R317: 1k, Resistor_SMD:R_0805_2012Metric_Pad1.15x1.40mm_HandSolder, B.Cu at (141.2, 67.2)
- added R318: 1k, Resistor_SMD:R_0805_2012Metric_Pad1.15x1.40mm_HandSolder, B.Cu at (141.3, 77.2)
- added R319: 1k, Resistor_SMD:R_0805_2012Metric_Pad1.15x1.40mm_HandSolder, B.Cu at (144.5, 128.2)
- added U401: 4011, Package_SO:SOIC-14_3.9x8.7mm_P1.27mm, B.Cu at (99.8, 87.2)
- J101, J102, J103, J104, J105, J302, J303, J304: footprint AJ-Dropbox-Kicad:AudioJack3StereoNarrow-PJ-321 -> Connector_Audio:Jack_3.5mm_Ledino_KB3SPRS_Horizontal
- R105, R311: value 100k -> OPEN
- RV101: footprint Potentiometer_THT:Potentiometer_Piher_T-16H_Double_Horizontal -> Potentiometer_THT:Potentiometer_Alps_RK163_Dual_Horizontal
- RV301: value 10k Sine -> 100k Freq
- moved R310 77.0 mm to (141.2, 141.5), turned to 0 degrees
- moved RV301 58.3 mm to (146.2, 77.2)
- moved R305 45.8 mm to (138.2, 119.5), turned to 90 degrees
- moved D303 45.7 mm to (133.2, 119.5), turned to 90 degrees
- moved D302 45.5 mm to (136.2, 119.5), turned to 270 degrees
- moved R304 35.5 mm to (133.2, 114.5), turned to 90 degrees
- moved R306 26.5 mm to (133.2, 110.0), turned to 270 degrees
- moved J303 22.0 mm to (144.2, 52.0)
- moved R309 19.6 mm to (145.0, 102.0), turned to 0 degrees
- moved C304 16.4 mm to (132.2, 89.0), turned to 90 degrees
- moved R307 15.0 mm to (145.0, 104.0), turned to 0 degrees
- moved R308 15.0 mm to (141.0, 102.0), turned to 0 degrees
- moved C305 13.9 mm to (132.0, 96.5), turned to 90 degrees
- moved R312 12.8 mm to (141.2, 72.2)
- moved R301 12.0 mm to (147.5, 108.5), turned to 180 degrees
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Connections:
- C102 pad 1: Charge -> Net-(C102-Pad1)
- C106 pad 1: Tri -> Net-(C106-Pad1)
- C303 pad 1: Tri3 -> Net-(C303-Pad1)
- R101 pad 2: Charge -> Net-(C102-Pad1)
- R103 pad 1: Square -> Charge
- R103 pad 2: Net-(R103-Pad2) -> Net-(C102-Pad1)
- R105 pad 2: Tri -> Net-(C106-Pad1)
- R108 pad 2: Sine -> Net-(R108-Pad2)
- R302 pad 2: Sine3 -> Net-(R302-Pad2)
- R310 pad 1: Net-(R310-Pad1) -> Net-(R302-Pad2)
- R310 pad 2: GND -> Sine3
- R311 pad 2: Tri3 -> Net-(C303-Pad1)
- RV101 pad 4: +12V -> Net-(R113-Pad1)
- RV301 pad 1: Net-(D302-Pad1) -> Net-(R318-Pad1)
- RV301 pad 2: Tri3 -> Square3fb
- RV301 pad 3: Tri3 -> Net-(R317-Pad2)
- SW101 pad 2: Charge -> Net-(C102-Pad1)
- U101 pad 2: Charge -> Net-(C102-Pad1)
- U101 pad 3: Net-(R103-Pad2) -> Net-(R114-Pad2)
- U101 pad 6: Charge -> Net-(C102-Pad1)
- U102 pad 1: Tri -> Net-(C106-Pad1)
- U102 pad 7: Sine -> Net-(R108-Pad2)
- U301 pad 1: Tri3 -> Net-(C303-Pad1)
- U301 pad 7: Sine3 -> Net-(R302-Pad2)
- U302 pad 6: Square3 -> Net-(R314-Pad2)
- U302 pad 7: Square3 -> Net-(R315-Pad2)
Routing:
- net Net-(D302-Pad1): track 75.3 -> 17.8 mm
- net Sine3: track 61.0 -> 4.57 mm
- net Net-(R302-Pad2): track 0.00 -> 52.3 mm
- net Net-(R315-Pad2): track 0.00 -> 41.5 mm
- net GND: track 306.6 -> 270.9 mm, vias 21 -> 37
- net Tri: track 36.6 -> 5.00 mm
- net Net-(C106-Pad1): track 0.00 -> 31.6 mm
- net Sine: track 23.4 -> 0.00 mm, vias 2 -> 0
- net Net-(R108-Pad2): track 0.00 -> 23.4 mm, vias 0 -> 2
- net Net-(C303-Pad1): track 0.00 -> 18.1 mm
- net Net-(R309-Pad2): track 53.5 -> 39.4 mm, vias 0 -> 2
- net Square3: track 14.2 -> 2.20 mm
- net Net-(R304-Pad2): track 21.5 -> 10.1 mm, vias 2 -> 0
- net Net-(U402-Pad12): track 11.1 -> 0.00 mm
- net Tri3: track 58.6 -> 47.7 mm, vias 2 -> 0
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- added copper zone on B.Cu, net GND
Other:
- board text added: "LFO1 Johansen Engineering 2019/10/01 - Rev 2A"
- board text removed: "LFO1 Johansen Engineering 2019/04/15 - Rev A"

Commit message: LFO 555 done
Parts:
- J103, J105: footprint Connector_Audio:Jack_3.5mm_Ledino_KB3SPRS_Horizontal -> AJ-Dropbox-Kicad:AudioJack3StereoNarrow-PJ-321
- R113, R114, R115, R116, R117: moved to B.Cu
- moved R115 100.0 mm to (60.2, 137.8), turned to 90 degrees
- moved R117 86.6 mm to (60.7, 123.0), turned to 180 degrees
- moved R116 79.8 mm to (51.0, 117.2), turned to 90 degrees
- moved R114 58.6 mm to (64.4, 100.2)
- moved R113 38.3 mm to (56.2, 73.3), turned to 90 degrees
- moved C101 34.0 mm to (53.2, 98.2), turned to 270 degrees
- moved C104 33.2 mm to (56.3, 141.8), turned to 180 degrees
- moved P101 26.5 mm to (65.2, 144.0), turned to 270 degrees
- moved C105 25.8 mm to (64.0, 141.8), turned to 180 degrees
- moved D103 24.9 mm to (66.5, 137.0)
- moved J105 23.0 mm to (55.2, 123.0)
- moved SW101 22.0 mm to (65.5, 78.7), turned to 0 degrees
- moved U101 21.9 mm to (59.2, 93.8), turned to 180 degrees
- moved C103 20.8 mm to (65.8, 70.8)
- moved U102 20.8 mm to (59.2, 115.8), turned to 180 degrees
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Routing:
- net Charge: track 59.6 -> 15.0 mm, vias 4 -> 0
- net Net-(C102-Pad1): track 0.00 -> 34.2 mm
- net Net-(C106-Pad2): track 44.0 -> 15.8 mm, vias 2 -> 0
- net Net-(R102-Pad1): track 25.7 -> 52.0 mm, vias 2 -> 0
- net Square: track 39.8 -> 14.8 mm
- net Net-(C106-Pad1): track 31.6 -> 55.1 mm
- net +12V: track 446.5 -> 467.6 mm, vias 3 -> 4
- net GND: track 270.9 -> 251.0 mm, vias 37 -> 41
- net Tri: track 5.00 -> 21.7 mm
- net Net-(R108-Pad2): track 23.4 -> 9.06 mm, vias 2 -> 0
- net -12V: track 244.6 -> 234.0 mm, vias 2 -> 0
- net Sine: track 0.00 -> 7.68 mm
- net Net-(R114-Pad2): track 0.00 -> 7.46 mm
- net Net-(R107-Pad2): track 12.9 -> 5.61 mm
- net Net-(C103-Pad1): track 9.61 -> 3.35 mm
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Other:
- board text added: "JE 555 LFO 1 2019/10/01 Rev 2A"
- board text added: "Rev 2A 2019/10/01 JE 555 LFO 1"
- board text removed: "JE 555 LFO 1 2019/03/19 Rev A"
- board text removed: "Johansen Engineering 2019/03/19 - Rev A 555 LFO 1"
